Commit message: Updated rs for new model

File: models/crawling_hand/crawling_hand_description/six_finger_hand_llll.urdf (robot description, URDF)
Before this commit: robot converted_robot, 63 links, 62 joints
Links:
- link MCP_motor_1: geometry visual mesh filename=package://converted_MCP_motor_1.stl; visual mesh filename=package://converted_proximal_1.stl
- link MCP_motor_2: geometry visual mesh filename=package://converted_MCP_motor_1.stl; visual mesh filename=package://converted_proximal_1.stl
- link MCP_motor_3: geometry visual mesh filename=package://converted_MCP_motor_1.stl; visual mesh filename=package://converted_proximal_1.stl
- link MCP_motor_4: geometry visual mesh filename=package://converted_MCP_motor_1.stl; visual mesh filename=package://converted_proximal_1.stl
- link MCP_motor_5: geometry visual mesh filename=package://converted_MCP_motor_1.stl; visual mesh filename=package://converted_proximal_1.stl
- link MCP_motor_6: geometry visual mesh filename=package://converted_MCP_motor_1.stl; visual mesh filename=package://converted_proximal_1.stl
- link MCP_spread_motor_1: geometry visual mesh filename=package://converted_MCP_spread_motor_1.stl; visual mesh filename=package://converted_metacarpal_1.stl
- link MCP_spread_motor_2: geometry visual mesh filename=package://converted_MCP_spread_motor_1.stl; visual mesh filename=package://converted_metacarpal_1.stl
- link MCP_spread_motor_3: geometry visual mesh filename=package://converted_MCP_spread_motor_1.stl; visual mesh filename=package://converted_metacarpal_1.stl
- link MCP_spread_motor_4: geometry visual mesh filename=package://converted_MCP_spread_motor_1.stl; visual mesh filename=package://converted_metacarpal_1.stl
- link MCP_spread_motor_5: geometry visual mesh filename=package://converted_MCP_spread_motor_1.stl; visual mesh filename=package://converted_metacarpal_1.stl
- link MCP_spread_motor_6: geometry visual mesh filename=package://converted_MCP_spread_motor_1.stl; visual mesh filename=package://converted_metacarpal_1.stl
- link PIP_DIP_motor_1: geometry visual mesh filename=package://converted_PIP_DIP_motor_1.stl; visual mesh filename=package://converted_middle_1.stl
- link PIP_DIP_motor_3: geometry visual mesh filename=package://converted_PIP_DIP_motor_1.stl; visual mesh filename=package://converted_middle_1.stl
- link PIP_DIP_motor_4: geometry visual mesh filename=package://converted_PIP_DIP_motor_1.stl; visual mesh filename=package://converted_middle_1.stl
- link PIP_DIP_motor_5: geometry visual mesh filename=package://converted_PIP_DIP_motor_1.stl; visual mesh filename=package://converted_middle_1.stl
- link PIP_DIP_motor_6: geometry visual mesh filename=package://converted_PIP_DIP_motor_1.stl; visual mesh filename=package://converted_middle_1.stl
- link PIP_DIP_motor__2: geometry visual mesh filename=package://converted_PIP_DIP_motor_1.stl; visual mesh filename=package://converted_middle_1.stl
- link distal_1: geometry visual mesh filename=package://converted_distal_1.stl
- link distal_2: geometry visual mesh filename=package://converted_distal_1.stl
- link distal_3: geometry visual mesh filename=package://converted_distal_1.stl
- link distal_4: geometry visual mesh filename=package://converted_distal_1.stl
- link distal_5: geometry visual mesh filename=package://converted_distal_1.stl
- link distal_6: geometry visual mesh filename=package://converted_distal_1.stl
- link finger_1: geometry visual mesh filename=package://converted_base_link.stl
- link finger_2: geometry visual mesh filename=package://converted_base_link.stl
- link finger_3: geometry visual mesh filename=package://converted_base_link.stl
- link finger_4: geometry visual mesh filename=package://converted_base_link.stl
- link finger_5: geometry visual mesh filename=package://converted_base_link.stl
- link finger_6: geometry visual mesh filename=package://converted_base_link.stl
- link hand: geometry visual box size=0.16 0.16 0.02

File: models/crawling_hand/single_finger/longest/URDF_finger_llll.urdf (robot description, URDF)
Before this commit: robot URDF_finger_llll, 8 links, 7 joints
Links:
- link MCP_motor_1: geometry collision mesh filename=package://longest/meshes/MCP_motor_1.stl scale=0.001 0.001 0.001; visual mesh filename=package://longest/meshes/MCP_motor_1.stl scale=0.001 0.001 0.001
- link MCP_spread_motor_1: geometry collision mesh filename=package://longest/meshes/MCP_spread_motor_1.stl scale=0.001 0.001 0.001; visual mesh filename=package://longest/meshes/MCP_spread_motor_1.stl scale=0.001 0.001 0.001
- link PIP_DIP_motor_1: geometry collision mesh filename=package://longest/meshes/PIP_DIP_motor_1.stl scale=0.001 0.001 0.001; visual mesh filename=package://longest/meshes/PIP_DIP_motor_1.stl scale=0.001 0.001 0.001
- link base_link: geometry collision mesh filename=package://longest/meshes/base_link.stl scale=0.001 0.001 0.001; visual mesh filename=package://longest/meshes/base_link.stl scale=0.001 0.001 0.001
- link distal_1: geometry collision mesh filename=package://longest/meshes/distal_1.stl scale=0.001 0.001 0.001; visual mesh filename=package://longest/meshes/distal_1.stl scale=0.001 0.001 0.001
- link metacarpal_1: geometry collision mesh filename=package://longest/meshes/metacarpal_1.stl scale=0.001 0.001 0.001; visual mesh filename=package://longest/meshes/metacarpal_1.stl scale=0.001 0.001 0.001
- link middle_1: geometry collision mesh filename=package://longest/meshes/middle_1.stl scale=0.001 0.001 0.001; visual mesh filename=package://longest/meshes/middle_1.stl scale=0.001 0.001 0.001
- link proximal_1: geometry collision mesh filename=package://longest/meshes/proximal_1.stl scale=0.001 0.001 0.001; visual mesh filename=package://longest/meshes/proximal_1.stl scale=0.001 0.001 0.001
Joints:
- joint DIP: limit (none) -> lower=-2.3 upper=2.3 effort=0 velocity=0
- joint MCP: limit (none) -> lower=-2.4 upper=2.4 effort=0 velocity=0
- joint MCP_spread: limit (none) -> lower=-1.9 upper=1.9 effort=0 velocity=0
- joint PIP: limit (none) -> lower=-2 upper=2 effort=0 velocity=0
