Commit message: Fixed finger urdf

File: models/crawling_hand/fingers/longest/URDF_finger_llll.urdf (robot description, URDF)
Before this commit: robot URDF_finger_llll, 8 links, 7 joints
Joints:
- joint DIP: limit lower=-2 upper=0. effort=0 velocity=0 -> lower=-2.3 upper=0. effort=0 velocity=0; origin xyz=0.003 0.0505 1.0 rpy=0 0 0 -> xyz=0.003 0.0505 0.0 rpy=0 0 0; type revolute -> continuous
- joint MCP: type revolute -> continuous
- joint MCP_spread: type revolute -> continuous
- joint PIP: type revolute -> continuous

Commit message: Added joint limits to the fingers

File: models/crawling_hand/fingers/longest/URDF_finger_llll.urdf (robot description, URDF)
Before this commit: robot URDF_finger_llll, 8 links, 7 joints
Joints:
- joint DIP: limit lower=-2.3 upper=0. effort=0 velocity=0 -> (none)
- joint MCP: limit lower=0 upper=2.4 effort=0 velocity=0 -> (none)
- joint MCP_spread: limit lower=-1.9 upper=1.9 effort=0 velocity=0 -> (none)
- joint PIP: limit lower=0 upper=2 effort=0 velocity=0 -> (none)

Commit message: Added limits and correct types for the fingers

File: models/crawling_hand/fingers/longest/URDF_finger_llll.urdf (robot description, URDF)
Before this commit: robot URDF_finger_llll, 8 links, 7 joints
Joints:
- joint DIP: limit (none) -> lower=-2.1 upper=0 effort=0 velocity=0; type continuous -> revolute
- joint MCP: limit (none) -> lower=0. upper=2. effort=0 velocity=0; type continuous -> revolute
- joint MCP_spread: limit (none) -> lower=-1.5 upper=1.5 effort=0 velocity=0; type continuous -> revolute
- joint PIP: limit (none) -> lower=0 upper=2.1 effort=0 velocity=0; type continuous -> revolute
