Commit message: Fixed hand model

File: models/crawling_hand/description/six_finger_hand_llll.urdf (robot description, URDF)
Before this commit: robot converted_robot, 63 links, 62 joints
Links:
- removed link MCP_spread_1
- removed link MCP_spread_2
- removed link MCP_spread_3
- removed link MCP_spread_4
- removed link MCP_spread_5
- removed link MCP_spread_6
- removed link hand2finger_1_fixed
- removed link hand2finger_2_fixed
- removed link hand2finger_3_fixed
- removed link hand2finger_4_fixed
- removed link hand2finger_5_fixed
- removed link hand2finger_6_fixed
- removed link world
- removed link world2world_fixed
Joints:
- removed joint MCP_spread_1_offset
- removed joint MCP_spread_2_offset
- removed joint MCP_spread_3_offset
- removed joint MCP_spread_4_offset
- removed joint MCP_spread_5_offset
- removed joint MCP_spread_6_offset
- removed joint hand2finger_1_fixed_offset
- removed joint hand2finger_2_fixed_offset
- removed joint hand2finger_3_fixed_offset
- removed joint hand2finger_4_fixed_offset
- removed joint hand2finger_5_fixed_offset
- removed joint hand2finger_6_fixed_offset
- removed joint world2world_fixed
- removed joint world2world_fixed_offset
- joint MCP_spread_1: child MCP_spread_1 -> MCP_spread_motor_1
- joint MCP_spread_2: child MCP_spread_2 -> MCP_spread_motor_2
- joint MCP_spread_3: child MCP_spread_3 -> MCP_spread_motor_3
- joint MCP_spread_4: child MCP_spread_4 -> MCP_spread_motor_4
- joint MCP_spread_5: child MCP_spread_5 -> MCP_spread_motor_5
- joint MCP_spread_6: child MCP_spread_6 -> MCP_spread_motor_6
- joint hand2finger_1_fixed: child hand2finger_1_fixed -> finger_1
- joint hand2finger_2_fixed: child hand2finger_2_fixed -> finger_2
- joint hand2finger_3_fixed: child hand2finger_3_fixed -> finger_3
- joint hand2finger_4_fixed: child hand2finger_4_fixed -> finger_4
- joint hand2finger_5_fixed: child hand2finger_5_fixed -> finger_5
- joint hand2finger_6_fixed: child hand2finger_6_fixed -> finger_6
